File: hardware/carrier/carrier.kicad_sch (KiCad schematic)
At the start: 82 parts, among them J1 PANEL+ / PANEL- (>=15 A, 4-6 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, J10 UART: 3V3 GND RX2(16) TX2(17), J11 5V / 5V SW / 3V3 / GND, J12 AUX + / - (>=15 A), J13 I2C: 3V3 GND SDA SCL, J14 ESP32 left row: EN,36,39,34,3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, J15 ESP32 right row: 23,22,1,3,21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, J2 BUCK IN + / -, J3 BUCK OUT + / - (set 5.0 V), J4 DS18B20: 3V3 / DATA / GND, J5 Optional 2nd probe, J6 Supercap 2.7 V 10 F (upper), J7 Supercap 2.7 V 10 F (lower), J8 microSD push-push with detect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, J9 Spare: 3V3 GND 32 33 36 26 27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, Q1 N-MOSFET >=60 V (>=100 V if D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, U1 DS3231SN (or RV-3028-C7, firm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, U2 INA180A3 (gain 100), U3 MCP1416 (or TC4427A class), U4 Load switch 5 V >=1 A, active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

Commit message: Carrier schematic draft-2: wired style (passives beside and wired to their pins, power symbols, labels only between blocks); netlist unchanged, verified net by net
Co-Authored-By: Claude Opus 5.5 <noreply@anthropic.com>
Claude-Session: https://claude.ai/code/session_01BMFMt5yCJVT3JQicJnUWqs
Parts:
- BT1: value CR2032 holder (no charging) -> CR2032
- C3: value 470u 10 V low ESR -> 470u 10V
- D0: value >=100 V >=15 A dual Schottky (e.g. 20 A 100 V) -> MBRB20100CT
- D1: value S3M (1000 V 3 A) -> S3M
- D2: value SMAJ5.0A (TVS, unidirectional) -> SMAJ5.0A
- D3: value ESD 3.3 V (e.g. PESD3V3L1BA) -> PESD3V3L1BA
- D4: value SS14 (flyback clamp) -> SS14
- D5: value Schottky >=100 V >=10 A (MBR10100 class) -> MBR10100
- D6: value DNP: SMCJ58A TVS (fit after bench test if needed) -> DNP: SMCJ58A
- F2: value PTC 0.5 A hold -> PTC 0.5 A
- F3: value PTC 0.2 A hold -> PTC 0.2 A
- F4: value ATO blade holder, fuse NOT fitted (<=3 A on v1; 9 A only with D5 heatsink) -> ATO holder, empty; now fitted
- J1: value PANEL+ / PANEL- (>=15 A, 4-6 mm2) -> PANEL+ / PANEL- (>=15 A)
- J10: value UART: 3V3 GND RX2(16) TX2(17) -> UART
- J13: value I2C: 3V3 GND SDA SCL -> I2C
- J14: value ESP32 left row: EN,36,39,34,35,32,33,25,26,27,14,12,13,GND,VIN -> ESP32 left row
- J15: value ESP32 right row: 23,22,1,3,21,19,18,5,17,16,4,2,15,GND,3V3 -> ESP32 right row
- J2: value BUCK IN + / - -> BUCK IN
- J3: value BUCK OUT + / - (set 5.0 V) -> BUCK OUT 5.0 V
- J4: value DS18B20: 3V3 / DATA / GND -> Probe 1
- J5: value Optional 2nd probe -> Probe 2
- J6: value Supercap 2.7 V 10 F (upper) -> Supercap 10 F (upper)
- J7: value Supercap 2.7 V 10 F (lower) -> Supercap 10 F (lower)
- J8: value microSD push-push with detect (Hirose DM3AT) -> microSD (Hirose DM3AT)
- J9: value Spare: 3V3 GND 32 33 36 26 27 13 14 -> Spare GPIO
- JP1: value Jumper: remove = sun sensor off -> Sun sensor on
- LED1: value Green, ~0.3 mA -> Green
- Q1: value N-MOSFET >=60 V (>=100 V if D6 fitted) >=20 A Rds(on)<=20 mOhm @4.5 V -> IRLR3110Z
- RSH1: value 5m 1% 2512 >=2 W -> 5m 1% 2512 3 W
- RSH2: value DNP (option: 2x 10m) -> DNP: 10m 2512
- U1: value DS3231SN (or RV-3028-C7, firmware change) -> DS3231SN
- U2: value INA180A3 (gain 100) -> INA180A3
- U3: value MCP1416 (or TC4427A class) -> MCP1416
- U4: value Load switch 5 V >=1 A, active-high EN, soft start (AP22804AW5 / TPS22918 class) -> AP22804AW5
Connections:
- net +5V_EXT: no longer names the net of F2.2, J11.1 (Pin_1)
- net 5V_SW: no longer names the net of C13.1, D4.1 (K), J11.2 (Pin_2), U4.1 (OUT)
- net AUX+: no longer names the net of D5.1 (K), J12.1 (Pin_1)
- net AUX_F: no longer names the net of D5.2 (A), F4.2
- net DQ_T: no longer names the net of D3.1 (A1), J4.2 (Pin_2), J5.2 (Pin_2), R12.1, R13.1, R20.1
- net GATE_IN: no longer names the net of JP1.2 (B), R5.1, U3.3 (IN)
- net ISENSE_RAW: no longer names the net of R6.1, U2.1
- net LED_A: no longer names the net of LED1.2 (A), R9.2
- net PV_F: no longer names the net of D1.2 (A), F1.2, R1.1
- net SHUNT_TOP: no longer names the net of Q1.3 (S), R21.2, RSH1.1, RSH2.1, U2.3 (+)
- net SW_EN: no longer names the net of R18.1, R19.2, U4.4 (EN)
- no-connect marks 10 -> 11
Other:
- note added: "1. SUN-SENSOR LOOP: J1 -> D0 -> Q1 -> RSH1 -> GND (drawn in block 1) Panel short-circuit current, ~1 ms every 10 s. Panel Isc 5.40 A (label), max ~6 A in cold strong sun. A vertical panel peaks near 1.8 A at noon. The panel cannot supply more than its Isc. 2. BOARD SUPPLY: PV+ -> F1 (2 A) -> D1 (3 A) -> buck -> +5V. Under 0.3 A. F1 and D1 are NOT in the measured path. 3. AUX (optional): PV+ -> F4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"
- note added: "2. Board supply"
- note added: "C8, C9: place at J8 pin 4 (VDD)"
- note added: "ESP32 module and Q1 gate"
- note added: "ISENSE (GPIO 35): RSH1 5 mOhm x INA180A3 gain 100 = 0.5 V/A. Range 0-6 A (pulsed); output clamps at 3.3 V (~6.6 A), harmless. U2 IN+ and IN- are Kelvin traces from the inner ends of RSH1's pads (drawn as separate wires from the shunt). VDIV (GPIO 34): R1 100k / R2 4k7 = x 22.3. Voc 44.5 V -> 2.00 V; 48 V -> 2.15 V; 60 V -> 2.69 V. Firmware DIVIDER = (100 + 4.7) / 4.7."
- note added: "PVA carrier board v1 - schematic draft-2 (wired). Generated from hardware/CARRIER.md via parts.py. Engineer review required before manufacture."
- note added: "Star ground: one point, at RSH1's GND end"
- note added: "The ESP32 is a complete ELEGOO dev board plugged into J14/J15: EN pull-up, buttons, USB-serial and strapping are on that board. EN and GPIO 0, 1, 2, 3, 12, 15 are not brought out. GPIO 5 (strapping) is held high by R14. Q1 gate: U3 drives it when +5V exists; R21 (100k, gate-source) holds Q1 off before that, at dawn. D6 (TVS on PV+): footprint only; fitted if the v1 bench test shows turn-off overs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"
- note added: "Wired style: each capacitor and resistor is drawn beside the pin it serves. +5V, +3V3 and GND are power symbols. Net labels only where a signal leaves its block. Placement priorities: PLACEMENT.md."
- note removed: "1. SUN-SENSOR LOOP: J1 -> D0 -> Q1 -> RSH1 -> GND Panel short-circuit current, ~1 ms every 10 s. Panel Isc 5.40 A (label), max ~6 A in cold strong sun. A vertical panel peaks near 1.8 A at noon. The panel cannot supply more than its Isc. 2. BOARD SUPPLY: PV+ -> F1 (2 A) -> D1 (3 A) -> buck -> +5V Under 0.3 A continuous. F1 and D1 are NOT in the measured current path: F1 sits after the Q1 node so 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"
- note removed: "2. Fuse, diode, divider"
- note removed: "ESP32 module and Q1 gate (review 2)"
- note removed: "ISENSE (GPIO 35): RSH1 5 mOhm x INA180A3 gain 100 = 0.5 V/A. Measured range 0-6 A (pulsed). 1.8 A -> 0.9 V; 5.4 A -> 2.7 V. Output clamps at the 3.3 V supply (~6.6 A): harmless. Gain 100 is deliberate: low vertical-panel currents stay well inside the ADC's range. Shunt dissipation 0.18 W only during each 1 ms pulse; 2 W rating is for pulse robustness. VDIV (GPIO 34): R1 100k / R2 4k7 = x 22.3 (R2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"
- note removed: "PVA carrier board v1 - schematic draft generated from hardware/CARRIER.md. Label style: nets join by name. Engineer review required before manufacture."
- note removed: "The ESP32 is a complete ELEGOO dev board plugged into J14/J15. Its EN pull-up, reset and boot buttons, USB-serial converter and strapping resistors are on that board, not on the carrier. EN and GPIO 0, 1, 2, 3, 12, 15 are deliberately not brought out. GPIO 5 (strapping) is held high by R14. Q1 gate: U3 drives it when +5V exists; R21 (100k, gate-source) holds Q1 off before that, at dawn. D6 (TVS o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"

Commit message: Carrier schematic: placement note for C3/C4 at ESP32 VIN
Co-Authored-By: Claude Opus 5.5 <noreply@anthropic.com>
Claude-Session: https://claude.ai/code/session_01BMFMt5yCJVT3JQicJnUWqs
Other:
- note added: "C3, C4: place at J14 pin 15 (ESP32 VIN)"
